Commit message: change friction paramter

File: urdf_xacro/macros_common_gazebo.urdf.xacro (robot description, xacro)
@@ -15,5 +15,5 @@
         </inertial>
     </xacro:macro>
-    <xacro:macro name="make_cylinder_collision" params="name:='collision' pose:=^|'0 0 0 0 0 0' length:=^ radius:=^ mu:=^|0.5 min_depth:=^|0.01">
+    <xacro:macro name="make_cylinder_collision" params="name:='collision' pose:=^|'0 0 0 0 0 0' length:=^ radius:=^ mu:=^|100.0 min_depth:=^|0.01">
         <collision name="${name}">
             <pose>${pose}</pose>
@@ -65,5 +65,5 @@
         </inertial>
     </xacro:macro>
-    <xacro:macro name="make_box_collision" params="name:='collision' pose:=^|'0 0 0 0 0 0' size:=^ mu:=^|0.5 min_depth:=^|0.01">
+    <xacro:macro name="make_box_collision" params="name:='collision' pose:=^|'0 0 0 0 0 0' size:=^ mu:=^|100.0 min_depth:=^|0.01">
         <collision name="${name}">
             <pose>${pose}</pose>
@@ -99,5 +99,5 @@
         </visual>
     </xacro:macro>
-    <xacro:macro name="make_polyline_collision" params="name:='collision' pose:=^|'0 0 0 0 0 0' **polyline mu:=^|0.5 min_depth:=^|0.01">
+    <xacro:macro name="make_polyline_collision" params="name:='collision' pose:=^|'0 0 0 0 0 0' **polyline mu:=^|100.0 min_depth:=^|0.01">
         <collision name="${name}">
             <pose>${pose}</pose>
@@ -134,5 +134,5 @@
     </xacro:macro>
     <!-- macros which expand to box/polyline collision and visual. convenient when defining pattern elements on a track -->
-    <xacro:macro name="make_box_element" params="pose:=^|'0 0 0 0 0 0' size:=^ mu:=^|0.5 min_depth:=^|0.01 *material">
+    <xacro:macro name="make_box_element" params="pose:=^|'0 0 0 0 0 0' size:=^ mu:=^|100.0 min_depth:=^|0.01 *material">
         <xacro:make_box_collision />
         <xacro:make_box_visual>
@@ -140,5 +140,5 @@
         </xacro:make_box_visual>
     </xacro:macro>
-    <xacro:macro name="make_polyline_element" params="pose:=^|'0 0 0 0 0 0' **polyline mu:=^|0.5 min_depth:=^|0.01 *material">
+    <xacro:macro name="make_polyline_element" params="pose:=^|'0 0 0 0 0 0' **polyline mu:=^|100.0 min_depth:=^|0.01 *material">
         <xacro:make_polyline_collision>
             <polyline>
@@ -185,5 +185,5 @@
     </xacro:macro>
     <!-- track segment templates which can be used with above population macros -->
-    <xacro:macro name="make_straight_segment_link_template" params="mass:=^ size_x:=^ size_y:=^ size_z:=^ mu:=^|0.5 min_depth:=^|0.01 *material">
+    <xacro:macro name="make_straight_segment_link_template" params="mass:=^ size_x:=^ size_y:=^ size_z:=^ mu:=^|100.0 min_depth:=^|0.01 *material">
         <xacro:make_box_inertial pose="${size_x / 2} 0 ${-size_z / 2} 0 0 0" />
         <xacro:make_box_collision pose="${size_x / 2} 0 ${-size_z / 2} 0 0 0" size="${size_x} ${size_y} ${size_z}" />
@@ -204,5 +204,5 @@
         </physics>
     </xacro:macro>
-    <xacro:macro name="make_arc_segment_link_template" params="mass:=^ length:=^ radius:=^ mu:=^|0.5 min_depth:=^|0.5 *material">
+    <xacro:macro name="make_arc_segment_link_template" params="mass:=^ length:=^ radius:=^ mu:=^|100.0 min_depth:=^|0.001 *material">
         <xacro:make_cylinder_inertial pose="0 0 ${-radius} ${pi / 2} 0 0" />
         <xacro:make_cylinder_collision pose="0 0 ${-radius} ${pi / 2} 0 0" />
@@ -225,5 +225,5 @@
     </xacro:macro>
     <!-- macros for populating track segments with above population macros and above templates -->
-    <xacro:macro name="populate_straight_segments" params="name_prefix:=^ x:=^|0 y:=^|0 z:=^|0 roll:=^|0 pitch:=^|0 yaw:=^|0 dx:=^|0 dy:=^|0 dz:=^|0 droll:=^|0 dpitch:=^|0 dyaw:=^|0 mass:=^ size_x:=^ size_y:=^ size_z:=^ parent:=^ mu:=^|0.5 min_depth:=^|0.01 implicit_spring_damper:=^|1 *material count:=^">
+    <xacro:macro name="populate_straight_segments" params="name_prefix:=^ x:=^|0 y:=^|0 z:=^|0 roll:=^|0 pitch:=^|0 yaw:=^|0 dx:=^|0 dy:=^|0 dz:=^|0 droll:=^|0 dpitch:=^|0 dyaw:=^|0 mass:=^ size_x:=^ size_y:=^ size_z:=^ parent:=^ mu:=^|100.0 min_depth:=^|0.01 implicit_spring_damper:=^|1 *material count:=^">
         <xacro:populate_links name_prefix="${name_prefix}_link">
             <template>
@@ -239,5 +239,5 @@
         </xacro:populate_joints>
     </xacro:macro>
-    <xacro:macro name="populate_arc_segments" params="name_prefix:=^ x:=^|0 y:=^|0 z:=^|0 roll:=^|0 pitch:=^|0 yaw:=^|0 dx:=^|0 dy:=^|0 dz:=^|0 droll:=^|0 dpitch:=^|0 dyaw:=^|0 mass:=^ length:=^ radius:=^ parent:=^ mu:=^|0.5 min_depth:=^|0.01 implicit_spring_damper:=^|1 *material count:=^">
+    <xacro:macro name="populate_arc_segments" params="name_prefix:=^ x:=^|0 y:=^|0 z:=^|0 roll:=^|0 pitch:=^|0 yaw:=^|0 dx:=^|0 dy:=^|0 dz:=^|0 droll:=^|0 dpitch:=^|0 dyaw:=^|0 mass:=^ length:=^ radius:=^ parent:=^ mu:=^|100.0 min_depth:=^|0.01 implicit_spring_damper:=^|1 *material count:=^">
         <xacro:populate_links name_prefix="${name_prefix}_link">
             <template>

File: urdf_xacro/macros_lugged_wheel_gazebo.urdf.xacro (robot description, xacro)
@@ -23,5 +23,5 @@
     </xacro:macro>
     <!-- main entry point: macro for making a lugged wheel by ContinuousTrack plugin -->
-    <xacro:macro name="make_lugged_wheel" params="name x:=^|0 y:=^|0 z:=^|0 roll:=^|0 pitch:=^|0 yaw:=^|0 mass:=^ radius:=^ width:=^ parent:=^ sprocket_joint:=^ pitch_diameter:=^ *material *pattern mu:=^|0.5 min_depth:=^|0.01 implicit_spring_damper:=^|1">
+    <xacro:macro name="make_lugged_wheel" params="name x:=^|0 y:=^|0 z:=^|0 roll:=^|0 pitch:=^|0 yaw:=^|0 mass:=^ radius:=^ width:=^ parent:=^ sprocket_joint:=^ pitch_diameter:=^ *material *pattern mu:=^|100.0 min_depth:=^|0.01 implicit_spring_damper:=^|1">
         <xacro:populate_arc_segments name_prefix="${name}_arc_segment" x="${x}" z="${z + radius}" mass="${mass / 4}" length="${width}" count="1">
             <xacro:insert_block name="material" />

File: urdf_xacro/macros_track_gazebo.urdf.xacro (robot description, xacro)
@@ -37,5 +37,5 @@
     </xacro:macro>
     <!-- main entry point: macro for making oval track by ContinuousTrack plugin -->
-    <xacro:macro name="make_track" params="name x:=^|0 y:=^|0 z:=^|0 roll:=^|0 pitch:=^|0 yaw:=^|0 mass:=^ length:=^ radius:=^ width:=^ parent:=^ sprocket_joint:=^ pitch_diameter:=^ *material *pattern mu:=^|0.5 min_depth:=^|0.01 implicit_spring_damper:=^|1">
+    <xacro:macro name="make_track" params="name x:=^|0 y:=^|0 z:=^|0 roll:=^|0 pitch:=^|0 yaw:=^|0 mass:=^ length:=^ radius:=^ width:=^ parent:=^ sprocket_joint:=^ pitch_diameter:=^ *material *pattern mu:=^|100.0 min_depth:=^|0.01 implicit_spring_damper:=^|1">
         <xacro:populate_straight_segments name_prefix="${name}_straight_segment" x="${x - length / 2}" z="${z + radius}" dx="${length}" dz="${-2 * radius}" dpitch="${pi}" mass="${mass / 4}" size_x="${length}" size_y="${width}" size_z="${radius}" count="2">
             <xacro:insert_block name="material" />

File: urdf_xacro/macros_track_simple_gazebo.urdf.xacro (robot description, xacro)
@@ -56,5 +56,5 @@
     </xacro:macro>
     <!-- main entry point: macro for making oval track by ContinuousTrackSimple plugin -->
-    <xacro:macro name="make_track_simple" params="name x:=^|0 y:=^|0 z:=^|0 roll:=^|0 pitch:=^|0 yaw:=^|0 mass:=^ length:=^ radius:=^ width:=^ parent:=^ sprocket_joint:=^ pitch_diameter:=^ mu:=^|0.5 min_depth:=^|0.01 implicit_spring_damper:=^|1 *material">
+    <xacro:macro name="make_track_simple" params="name x:=^|0 y:=^|0 z:=^|0 roll:=^|0 pitch:=^|0 yaw:=^|0 mass:=^ length:=^ radius:=^ width:=^ parent:=^ sprocket_joint:=^ pitch_diameter:=^ mu:=^|100.0 min_depth:=^|0.01 implicit_spring_damper:=^|1 *material">
         <xacro:populate_straight_segments name_prefix="${name}_straight_segment" x="${x - length / 2}" z="${z + radius}" dx="${length}" dz="${-2 * radius}" dpitch="${pi}" mass="${mass / 4}" size_x="${length}" size_y="${width}" size_z="${radius}" count="2">
             <xacro:insert_block name="material" />
@@ -65,5 +65,5 @@
         <xacro:make_track_simple_plugin name="${name}" />
     </xacro:macro>
-    <xacro:macro name="make_track_simple_wheels" params="name x:=^|0 y:=^|0 z:=^|0 roll:=^|0 pitch:=^|0 yaw:=^|0 mass:=^ length:=^ radius:=^ width:=^ parent:=^ sprocket_joint:=^ pitch_diameter:=^ mu:=^|0.5 min_depth:=^|0.01 implicit_spring_damper:=^|1 *material count:=^">
+    <xacro:macro name="make_track_simple_wheels" params="name x:=^|0 y:=^|0 z:=^|0 roll:=^|0 pitch:=^|0 yaw:=^|0 mass:=^ length:=^ radius:=^ width:=^ parent:=^ sprocket_joint:=^ pitch_diameter:=^ mu:=^|100.0 min_depth:=^|0.01 implicit_spring_damper:=^|1 *material count:=^">
         <xacro:populate_arc_segments name_prefix="${name}_wheel" x="${x + length / 2}"  z="${z + radius}" dx="${-length / (count - 1)}" mass="${mass / count}" length="${width}">
             <xacro:insert_block name="material" />
